Commit message: Fix: bridge camera node

File: src/tunnel_inspection_sim/urdf/tunnel_robot.xacro (robot description, xacro)
@@ -57,16 +57,34 @@
     <origin xyz="0.1 0 0.08" rpy="0 0 0"/>
   </joint>
-  <link name="left_camera_link"/>
   <joint name="left_camera_joint" type="fixed">
+    <origin xyz="0.1 0.05 0.1" rpy="0 -0.8 0.785"/>
     <parent link="base_link"/>
     <child link="left_camera_link"/>
-    <origin xyz="0.1 0.05 0.1" rpy="0 -0.5 0.785"/>
   </joint>
-  <link name="right_camera_link"/>
+  <link name="left_camera_link">
+    <visual>
+      <geometry><box size="0.01 0.01 0.01"/></geometry>
+      <material name="dark_gray"><color rgba="0.2 0.2 0.2 1.0"/></material>
+    </visual>
+    <inertial>
+      <mass value="0.001"/>
+      <inertia ixx="0.00001" ixy="0" ixz="0" iyy="0.00001" iyz="0" izz="0.00001"/>
+    </inertial>
+  </link>
   <joint name="right_camera_joint" type="fixed">
+    <origin xyz="0.1 -0.05 0.1" rpy="0 -0.8 -0.785"/>
     <parent link="base_link"/>
     <child link="right_camera_link"/>
-    <origin xyz="0.1 -0.05 0.1" rpy="0 -0.5 -0.785"/>
   </joint>
+  <link name="right_camera_link">
+    <visual>
+      <geometry><box size="0.01 0.01 0.01"/></geometry>
+      <material name="dark_gray"><color rgba="0.2 0.2 0.2 1.0"/></material>
+    </visual>
+    <inertial>
+      <mass value="0.001"/>
+      <inertia ixx="0.00001" ixy="0" ixz="0" iyy="0.00001" iyz="0" izz="0.00001"/>
+    </inertial>
+  </link>
   <gazebo>
     <plugin filename="libignition-gazebo-diff-drive-system.so" name="ignition::gazebo::systems::DiffDrive">
@@ -111,12 +129,19 @@
   <gazebo reference="left_camera_link">
     <sensor name="left_rgbd_camera" type="rgbd_camera">
-      <topic>left_camera</topic>
-      <update_rate>15</update_rate>
+      <topic>/left_camera</topic>
+      <gz_frame_id>left_camera_link</gz_frame_id>
+      <update_rate>15.0</update_rate>
       <camera>
         <horizontal_fov>1.047</horizontal_fov>
-        <image><width>640</width><height>480</height></image>
-        <clip><near>0.1</near><far>10.0</far></clip>
+        <image>
+          <width>640</width>
+          <height>480</height>
+        </image>
+        <clip>
+          <near>0.1</near>
+          <far>10.0</far>
+        </clip>
       </camera>
-      <always_on>1</always_on>
+      <always_on>true</always_on>
       <visualize>true</visualize>
     </sensor>
@@ -124,12 +149,19 @@
   <gazebo reference="right_camera_link">
     <sensor name="right_rgbd_camera" type="rgbd_camera">
-      <topic>right_camera</topic>
-      <update_rate>15</update_rate>
+      <topic>/right_camera</topic>
+      <gz_frame_id>right_camera_link</gz_frame_id>
+      <update_rate>15.0</update_rate>
       <camera>
         <horizontal_fov>1.047</horizontal_fov>
-        <image><width>640</width><height>480</height></image>
-        <clip><near>0.1</near><far>10.0</far></clip>
+        <image>
+          <width>640</width>
+          <height>480</height>
+        </image>
+        <clip>
+          <near>0.1</near>
+          <far>10.0</far>
+        </clip>
       </camera>
-      <always_on>1</always_on>
+      <always_on>true</always_on>
       <visualize>true</visualize>
     </sensor>

Commit message: Crack marker mapping 위치 수정

File: src/tunnel_inspection_sim/urdf/tunnel_robot.xacro (robot description, xacro)
@@ -72,4 +72,10 @@
     </inertial>
   </link>
+  <joint name="left_camera_optical_joint" type="fixed">
+    <origin xyz="0 0 0" rpy="-1.5708 0 -1.5708"/>
+    <parent link="left_camera_link"/>
+    <child link="left_camera_optical_frame"/>
+  </joint>
+  <link name="left_camera_optical_frame"/>
   <joint name="right_camera_joint" type="fixed">
     <origin xyz="0.1 -0.05 0.1" rpy="0 -0.8 -0.785"/>
@@ -87,4 +93,10 @@
     </inertial>
   </link>
+  <joint name="right_camera_optical_joint" type="fixed">
+    <origin xyz="0 0 0" rpy="-1.5708 0 -1.5708"/>
+    <parent link="right_camera_link"/>
+    <child link="right_camera_optical_frame"/>
+  </joint>
+  <link name="right_camera_optical_frame"/>
   <gazebo>
     <plugin filename="libignition-gazebo-diff-drive-system.so" name="ignition::gazebo::systems::DiffDrive">
@@ -130,5 +142,5 @@
     <sensor name="left_rgbd_camera" type="rgbd_camera">
       <topic>/left_camera</topic>
-      <gz_frame_id>left_camera_link</gz_frame_id>
+      <gz_frame_id>left_camera_optical_frame</gz_frame_id>
       <update_rate>15.0</update_rate>
       <camera>
@@ -150,5 +162,5 @@
     <sensor name="right_rgbd_camera" type="rgbd_camera">
       <topic>/right_camera</topic>
-      <gz_frame_id>right_camera_link</gz_frame_id>
+      <gz_frame_id>right_camera_optical_frame</gz_frame_id>
       <update_rate>15.0</update_rate>
       <camera>

Commit message: 카메라 pitch 10도씩 낮춤

File: src/tunnel_inspection_sim/urdf/tunnel_robot.xacro (robot description, xacro)
@@ -58,5 +58,5 @@
   </joint>
   <joint name="left_camera_joint" type="fixed">
-    <origin xyz="0.1 0.05 0.1" rpy="0 -0.55 1.05"/>
+    <origin xyz="0.1 0.05 0.1" rpy="0 -0.3755 1.05"/>
     <parent link="base_link"/>
     <child link="left_camera_link"/>
@@ -79,5 +79,5 @@
   <link name="left_camera_optical_frame"/>
   <joint name="top_camera_joint" type="fixed">
-    <origin xyz="0.1 0 0.12" rpy="0 -1.45 0"/>
+    <origin xyz="0.1 0 0.12" rpy="0 -1.2755 0"/>
     <parent link="base_link"/>
     <child link="top_camera_link"/>
@@ -100,5 +100,5 @@
   <link name="top_camera_optical_frame"/>
   <joint name="right_camera_joint" type="fixed">
-    <origin xyz="0.1 -0.05 0.1" rpy="0 -0.55 -1.05"/>
+    <origin xyz="0.1 -0.05 0.1" rpy="0 -0.3755 -1.05"/>
     <parent link="base_link"/>
     <child link="right_camera_link"/>

Commit message: 카메라 pitch 5도씩 더 낮춤

File: src/tunnel_inspection_sim/urdf/tunnel_robot.xacro (robot description, xacro)
@@ -58,5 +58,5 @@
   </joint>
   <joint name="left_camera_joint" type="fixed">
-    <origin xyz="0.1 0.05 0.1" rpy="0 -0.3755 1.05"/>
+    <origin xyz="0.1 0.05 0.1" rpy="0 -0.2882 1.05"/>
     <parent link="base_link"/>
     <child link="left_camera_link"/>
@@ -79,5 +79,5 @@
   <link name="left_camera_optical_frame"/>
   <joint name="top_camera_joint" type="fixed">
-    <origin xyz="0.1 0 0.12" rpy="0 -1.2755 0"/>
+    <origin xyz="0.1 0 0.12" rpy="0 -1.1882 0"/>
     <parent link="base_link"/>
     <child link="top_camera_link"/>
@@ -100,5 +100,5 @@
   <link name="top_camera_optical_frame"/>
   <joint name="right_camera_joint" type="fixed">
-    <origin xyz="0.1 -0.05 0.1" rpy="0 -0.3755 -1.05"/>
+    <origin xyz="0.1 -0.05 0.1" rpy="0 -0.2882 -1.05"/>
     <parent link="base_link"/>
     <child link="right_camera_link"/>
